File: pcb/dice.brd (EAGLE design)
At the start: 55.9 x 48.3 mm, 23 parts

Commit message: Minor changes
Parts:
- renumbered E$1 to D3, E$10 to D8, E$11 to D11, E$12 to D12, E$13 to D13, E$14 to D14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
Other:
- board text added: "Electronic Dice R2 (c) afiskon 2017"
- board text removed: "PB0"
- board text removed: "PB1"
- board text removed: "PB2"
- board text removed: "PB3"
- board text removed: "afiskon'17"
